File: todd/hardware/todd_watch.kicad_pcb (KiCad board)
At the start: 0 parts

Commit message: Schem 1 done
Parts:
- added AE1: Bluetooth, RF_Antenna:Texas_SWRA117D_2.4GHz_Left, F.Cu at (97.8, 88.7)
- added AE2: NFC Stub, Resistor_SMD:R_1206_3216Metric_Pad1.30x1.75mm_HandSolder, F.Cu at (138.7, 84.2)
- added BT1: Pouch, Connector_PinSocket_2.54mm:PinSocket_1x02_P2.54mm_Vertical, F.Cu at (118.3, 110.5)
- added BT2: Cell, Battery:BatteryHolder_Keystone_1042_1x18650, F.Cu at (129.2, 71.2)
- added C1: 4.7u, Capacitor_SMD:C_0603_1608Metric, F.Cu at (135.9, 111.4)
- added C10: 1u, Capacitor_SMD:C_0603_1608Metric, F.Cu at (154.3, 93.8)
- added C11: 2.2u, Capacitor_SMD:C_0603_1608Metric, F.Cu at (142.7, 92.9)
- added C12: 820p, Capacitor_SMD:C_0603_1608Metric, F.Cu at (135.9, 116.4)
- added C13: Z1, Capacitor_SMD:C_0603_1608Metric, F.Cu at (133.0, 104.8)
- added C14: 1u, Capacitor_SMD:C_0603_1608Metric, F.Cu at (141.1, 106.4)
- added C15: 100n, Capacitor_SMD:C_0603_1608Metric, F.Cu at (139.9, 111.4)
- added C16: 100n, Capacitor_SMD:C_0603_1608Metric, F.Cu at (127.9, 112.3)
- added C17: 100n, Capacitor_SMD:C_0603_1608Metric, F.Cu at (131.9, 109.8)
- added C18: 100n, Capacitor_SMD:C_0603_1608Metric, F.Cu at (158.3, 86.3)
- added C19: 100n, Capacitor_SMD:C_0603_1608Metric, F.Cu at (133.0, 107.3)
- added C2: 4.7u, Capacitor_SMD:C_0603_1608Metric, F.Cu at (150.2, 98.8)
- added C20: 100n, Capacitor_SMD:C_0603_1608Metric, F.Cu at (123.0, 117.8)
- added C21: 100n, Capacitor_SMD:C_0603_1608Metric, F.Cu at (98.3, 107.9)
- added C22: 100n, Capacitor_SMD:C_0603_1608Metric, F.Cu at (126.0, 99.8)
- added C23: 1u, Capacitor_SMD:C_0603_1608Metric, F.Cu at (130.0, 102.3)
- added C24: 1u, Capacitor_SMD:C_0603_1608Metric, F.Cu at (135.9, 113.9)
- added C25: 1u, Capacitor_SMD:C_0603_1608Metric, F.Cu at (129.0, 104.8)
- added C26: 0.1u, Capacitor_SMD:C_0603_1608Metric, F.Cu at (162.3, 91.3)
- added C27: 27n, Capacitor_SMD:C_0603_1608Metric, F.Cu at (141.1, 103.9)
- added C28: 10u, Capacitor_SMD:C_0603_1608Metric, F.Cu at (86.9, 123.1)
- added C29: 1u, Capacitor_SMD:C_0603_1608Metric, F.Cu at (123.0, 115.3)
- added C3: 100p, Capacitor_SMD:C_0603_1608Metric, F.Cu at (134.0, 101.5)
- added C30: 10u, Capacitor_SMD:C_0603_1608Metric, F.Cu at (105.1, 117.8)
- added C31: 1u, Capacitor_SMD:C_0603_1608Metric, F.Cu at (163.7, 88.8)
- added C32: 10u, Capacitor_SMD:C_0603_1608Metric, F.Cu at (102.3, 107.9)
- added C33: 1u, Capacitor_SMD:C_0603_1608Metric, F.Cu at (131.9, 116.4)
- added C34: 10u, Capacitor_SMD:C_0603_1608Metric, F.Cu at (109.6, 101.6)
- added C35: 10u, Capacitor_SMD:C_0603_1608Metric, F.Cu at (138.2, 97.0)
- added C36: 1u, Capacitor_SMD:C_0603_1608Metric, F.Cu at (150.2, 101.3)
- added C37: 1u, Capacitor_SMD:C_0603_1608Metric, F.Cu at (129.0, 107.3)
- added C38: 27p, Capacitor_SMD:C_0603_1608Metric, F.Cu at (113.6, 101.6)
- added C39: 27p, Capacitor_SMD:C_0603_1608Metric, F.Cu at (134.2, 96.4)
- added C4: 2.2u, Capacitor_SMD:C_0603_1608Metric, F.Cu at (151.7, 88.8)
- added C40: 100n, Capacitor_SMD:C_0603_1608Metric, F.Cu at (145.1, 103.9)
- added C41: 100n, Capacitor_SMD:C_0603_1608Metric, F.Cu at (137.1, 104.0)
- added C42: 100n, Capacitor_SMD:C_0603_1608Metric, F.Cu at (157.0, 83.8)
- added C43: 100n, Capacitor_SMD:C_0603_1608Metric, F.Cu at (147.6, 88.8)
- added C44: 100n, Capacitor_SMD:C_0603_1608Metric, F.Cu at (146.7, 93.8)
- added C45: 100n, Capacitor_SMD:C_0603_1608Metric, F.Cu at (142.2, 100.4)
- added C46: 100n, Capacitor_SMD:C_0603_1608Metric, F.Cu at (187.2, 73.2)
- added C47: 100n, Capacitor_SMD:C_0603_1608Metric, F.Cu at (116.8, 121.7)
- added C48: 2.2u, Capacitor_SMD:C_0603_1608Metric, F.Cu at (142.2, 97.9)
- added C49: 2.2u, Capacitor_SMD:C_0603_1608Metric, F.Cu at (90.9, 123.1)
- added C5: Z3, Capacitor_SMD:C_0603_1608Metric, F.Cu at (154.3, 98.8)
- added C50: 100n, Capacitor_SMD:C_0603_1608Metric, F.Cu at (126.0, 102.3)
- added C51: 100n, Capacitor_SMD:C_0603_1608Metric, F.Cu at (134.2, 98.9)
- added C52: 100n, Capacitor_SMD:C_0603_1608Metric, F.Cu at (153.0, 86.3)
- added C53: 100n, Capacitor_SMD:C_0603_1608Metric, F.Cu at (162.3, 86.3)
- added C6: 1u, Capacitor_SMD:C_0603_1608Metric, F.Cu at (146.2, 101.3)
- added C7: 1u, Capacitor_SMD:C_0603_1608Metric, F.Cu at (127.9, 109.8)
- added C8: 100n, Capacitor_SMD:C_0603_1608Metric, F.Cu at (130.0, 99.8)
- added C9: 1u, Capacitor_SMD:C_0603_1608Metric, F.Cu at (109.1, 117.8)
- added J1: Expansion, Connector_PinSocket_1.27mm:PinSocket_2x09_P1.27mm_Vertical, F.Cu at (176.7, 61.5)
- added J3: LRA, Connector_PinHeader_2.54mm:PinHeader_1x02_P2.54mm_Vertical, F.Cu at (113.6, 114.2)
- added J4: USB Program, Connector_USB:USB_C_Receptacle_XKB_U262-16XN-4BVC11, F.Cu at (179.4, 78.6)
- added J5: FTDI Flash, Connector_PinHeader_1.27mm:PinHeader_1x05_P1.27mm_Vertical, F.Cu at (119.2, 90.9)
- added J6: Strap, Connector_PinHeader_2.54mm:PinHeader_1x04_P2.54mm_Vertical, F.Cu at (103.9, 84.8)
- added J7: Display, Connector_FFC-FPC:Hirose_FH12-10S-0.5SH_1x10-1MP_P0.50mm_Horizontal, F.Cu at (91.0, 93.2)
- added JP1: CPU VBus Power, Connector_PinHeader_1.27mm:PinHeader_2x01_P1.27mm_Horizontal, F.Cu at (118.4, 84.2)
- added JP10: Master 3.0v, Connector_PinHeader_1.27mm:PinHeader_1x02_P1.27mm_Horizontal, F.Cu at (131.1, 88.3)
- added JP11: Display 1.8v Power, Connector_PinHeader_1.27mm:PinHeader_1x02_P1.27mm_Horizontal, F.Cu at (104.8, 113.5)
- added JP12: IMU Address, Jumper:SolderJumper-3_P2.0mm_Open_TrianglePad1.0x1.5mm_NumberLabels, F.Cu at (182.1, 70.2)
- added JP13: Display Light Power, Connector_PinHeader_1.27mm:PinHeader_1x02_P1.27mm_Horizontal, F.Cu at (125.7, 95.5)
- added JP14: Display 3.0v Power, Connector_PinHeader_1.27mm:PinHeader_1x02_P1.27mm_Horizontal, F.Cu at (104.3, 121.3)
- added JP15: ALS Power, Connector_PinHeader_1.27mm:PinHeader_1x02_P1.27mm_Horizontal, F.Cu at (122.9, 90.9)
- added JP16: Mic Power, Connector_PinHeader_1.27mm:PinHeader_1x02_P1.27mm_Horizontal, F.Cu at (190.8, 61.5)
- added JP17: IMU Power, Connector_PinHeader_1.27mm:PinHeader_1x02_P1.27mm_Horizontal, F.Cu at (96.1, 121.3)
- added JP18: Flash Power, Connector_PinHeader_1.27mm:PinHeader_1x02_P1.27mm_Horizontal, F.Cu at (116.5, 105.2)
- added JP2: CPU HiVolt, Connector_PinHeader_1.27mm:PinHeader_2x01_P1.27mm_Horizontal, F.Cu at (127.9, 85.0)
- added JP3: CPU 1.8v Power, Connector_PinHeader_1.27mm:PinHeader_2x01_P1.27mm_Horizontal, F.Cu at (86.6, 120.2)
- added JP4: Haptic Ground, Jumper:SolderJumper-2_P1.3mm_Open_TrianglePad1.0x1.5mm, F.Cu at (134.4, 93.4)
- added JP5: I2C Power, Connector_PinHeader_1.27mm:PinHeader_2x01_P1.27mm_Horizontal, F.Cu at (97.9, 105.0)
- added JP6: Button Power, Connector_PinHeader_1.27mm:PinHeader_2x01_P1.27mm_Horizontal, F.Cu at (118.4, 87.5)
- added JP7: Cell Select, Connector_PinHeader_1.27mm:PinHeader_1x03_P1.27mm_Horizontal, F.Cu at (117.5, 99.3)
- added JP8: Power Select, Connector_PinHeader_1.27mm:PinHeader_1x03_P1.27mm_Horizontal, F.Cu at (109.3, 96.1)
- added JP9: Master 1.8v, Connector_PinHeader_1.27mm:PinHeader_2x01_P1.27mm_Horizontal, F.Cu at (109.3, 92.8)
- added L1: Z2, Inductor_SMD:L_0603_1608Metric, F.Cu at (146.2, 97.9)
- added L10: 4.7u, Inductor_SMD:L_0603_1608Metric, F.Cu at (154.3, 96.3)
- added L2: 10u, Inductor_SMD:L_0603_1608Metric, F.Cu at (187.7, 69.6)
- added L3: 10u, Inductor_SMD:L_0603_1608Metric, F.Cu at (138.2, 99.5)
- added L4: 15n, Inductor_SMD:L_0603_1608Metric, F.Cu at (155.7, 88.8)
- added L5: 15n, Inductor_SMD:L_0603_1608Metric, F.Cu at (150.2, 96.3)
- added L6: 10u, Inductor_SMD:L_0603_1608Metric, F.Cu at (127.9, 114.8)
- added L7: 2.2u, Inductor_SMD:L_0603_1608Metric, F.Cu at (137.1, 108.9)
- added L8: 2.2u, Inductor_SMD:L_0603_1608Metric, F.Cu at (147.6, 91.3)
- added L9: 4.7u, Inductor_SMD:L_0603_1608Metric, F.Cu at (153.0, 83.8)
- added MK1: ICS-40619, parts:MIC_ICS-40619, F.Cu at (118.7, 117.9)
- added R1: 4.7, Resistor_SMD:R_0603_1608Metric, F.Cu at (125.0, 104.8)
- added R10: 10k, Resistor_SMD:R_0603_1608Metric, F.Cu at (154.3, 91.3)
- added R11: 470, Resistor_SMD:R_0603_1608Metric, F.Cu at (120.8, 121.7)
- added R12: 47k, Resistor_SMD:R_0603_1608Metric, F.Cu at (159.7, 88.8)
- added R13: 10k, Resistor_SMD:R_0603_1608Metric, F.Cu at (162.3, 83.8)
- added R14: 10k, Resistor_SMD:R_0603_1608Metric, F.Cu at (145.1, 106.4)
- added R2: ???, Resistor_SMD:R_0603_1608Metric, F.Cu at (149.1, 103.9)
- added R3: 47k, Resistor_SMD:R_0603_1608Metric, F.Cu at (158.3, 93.8)
- added R4: 10k, Resistor_SMD:R_0603_1608Metric, F.Cu at (166.3, 83.8)
- added R5: 47k, Resistor_SMD:R_0603_1608Metric, F.Cu at (142.7, 95.4)
- added R6: ???, Resistor_SMD:R_0603_1608Metric, F.Cu at (166.3, 86.3)
- added R7: 5.1k, Resistor_SMD:R_0603_1608Metric, F.Cu at (127.1, 118.9)
- added R8: 5.1k, Resistor_SMD:R_0603_1608Metric, F.Cu at (141.1, 108.9)
- added R9: 12k 1%, Resistor_SMD:R_0603_1608Metric, F.Cu at (131.9, 113.9)
- added SW1: Up, Button_Switch_THT:SW_PUSH_6mm, F.Cu at (99.1, 96.8)
- added SW2: Select, Button_Switch_THT:SW_PUSH_6mm, F.Cu at (86.9, 112.0)
- added SW3: Down, Button_Switch_THT:SW_PUSH_6mm, F.Cu at (180.7, 61.8)
- added SW4: Back, Button_Switch_THT:SW_PUSH_6mm, F.Cu at (108.2, 84.5)
- added TH1: ???, Capacitor_SMD:C_0603_1608Metric, F.Cu at (158.3, 91.3)
- added TP1: SPI Data In, TestPoint:TestPoint_Pad_D1.0mm, F.Cu at (175.9, 84.8)
- added TP10: I2C Data, TestPoint:TestPoint_Pad_D1.0mm, F.Cu at (128.0, 122.0)
- added TP11: Sys Tap, TestPoint:TestPoint_Pad_D1.0mm, F.Cu at (154.7, 104.7)
- added TP12: HV LDO Tap, TestPoint:TestPoint_Pad_D1.0mm, F.Cu at (148.6, 109.7)
- added TP13: LV LDO Tap, TestPoint:TestPoint_Pad_D1.0mm, F.Cu at (186.7, 76.0)
- added TP14: Buck 1 Tap, TestPoint:TestPoint_Pad_D1.0mm, F.Cu at (148.6, 106.6)
- added TP15: Buck 2 Tap, TestPoint:TestPoint_Pad_D1.0mm, F.Cu at (190.7, 66.0)
- added TP16: Charge Pump Tap, TestPoint:TestPoint_Pad_D1.0mm, F.Cu at (193.8, 66.0)
- added TP17: Boost Tap, TestPoint:TestPoint_Pad_D1.0mm, F.Cu at (165.8, 91.6)
- added TP18: Buck Boost Tap, TestPoint:TestPoint_Pad_D1.0mm, F.Cu at (139.4, 114.2)
- added TP19: Smartstrap Data, TestPoint:TestPoint_Pad_D1.0mm, F.Cu at (169.8, 84.0)
- added TP2: Safe Tap, TestPoint:TestPoint_Pad_D1.0mm, F.Cu at (172.9, 84.8)
- added TP20: Hivolt SWDCLK, TestPoint:TestPoint_Pad_D1.0mm, F.Cu at (163.9, 94.6)
- added TP21: Hivolt SWDIO, TestPoint:TestPoint_Pad_D1.0mm, F.Cu at (145.6, 109.2)
- added TP22: Hivolt RESET, TestPoint:TestPoint_Pad_D1.0mm, F.Cu at (160.8, 96.6)
- added TP23: Spare Shift 3.3v, TestPoint:TestPoint_Pad_D1.0mm, F.Cu at (142.5, 117.2)
- added TP24: Spare Shift 1.8v, TestPoint:TestPoint_Pad_D1.0mm, F.Cu at (159.9, 99.7)
- added TP25: Lovolt SWDCLK, TestPoint:TestPoint_Pad_D1.0mm, F.Cu at (168.9, 93.2)
- added TP26: Lovolt SWDIO, TestPoint:TestPoint_Pad_D1.0mm, F.Cu at (131.0, 122.0)
- added TP27: Lovolt RESET, TestPoint:TestPoint_Pad_D1.0mm, F.Cu at (151.7, 106.6)
- added TP28: LED One Sink, TestPoint:TestPoint_Pad_D1.0mm, F.Cu at (171.9, 90.2)
- added TP29: LED Two Sink, TestPoint:TestPoint_Pad_D1.0mm, F.Cu at (157.8, 96.6)
- added TP3: Power MPC1, TestPoint:TestPoint_Pad_D1.0mm, F.Cu at (137.1, 122.0)
- added TP30: Microphone Positive, TestPoint:TestPoint_Pad_D1.0mm, F.Cu at (145.6, 112.2)
- added TP31: Microphone Negative, TestPoint:TestPoint_Pad_D1.0mm, F.Cu at (153.8, 101.6)
- added TP4: Power MPC3, TestPoint:TestPoint_Pad_D1.0mm, F.Cu at (156.8, 101.6)
- added TP5: Power LED 2, TestPoint:TestPoint_Pad_D1.0mm, F.Cu at (134.1, 122.0)
- added TP6: Power MPC0, TestPoint:TestPoint_Pad_D1.0mm, F.Cu at (169.8, 87.1)
- added TP7: Power MPC2, TestPoint:TestPoint_Pad_D1.0mm, F.Cu at (168.9, 90.2)
- added TP8: Power MPC4, TestPoint:TestPoint_Pad_D1.0mm, F.Cu at (139.4, 117.2)
- added TP9: I2C Clock, TestPoint:TestPoint_Pad_D1.0mm, F.Cu at (142.5, 114.2)
- added U1: NRF5340-QKAA-AB0-R, parts:XCVR_NRF5340-QKAA-AB0-R, F.Cu at (110.5, 107.6)
- added U10: S25FS512SDSBHV210, parts:S25FL512SAGBHIC10, F.Cu at (99.3, 114.8)
- added U11: Si1151-AB00, si1151:10-WFQFN, F.Cu at (138.8, 93.9)
- added U2: MAX20353AEWN+, parts:MAX20353AEWN&plus_, F.Cu at (123.2, 111.1)
- added U3: FT232H, Package_QFP:LQFP-48_7x7mm_P0.5mm, F.Cu at (90.6, 104.2)
- added U4: TXS0102YZP, Package_BGA:Texas_DSBGA-8_0.9x1.9mm_Layout2x4_P0.5mm, F.Cu at (143.6, 89.1)
- added U5: TXS0102YZP, Package_BGA:Texas_DSBGA-8_0.9x1.9mm_Layout2x4_P0.5mm, F.Cu at (149.0, 85.0)
- added U6: TXS0102YZP, Package_BGA:Texas_DSBGA-8_0.9x1.9mm_Layout2x4_P0.5mm, F.Cu at (139.7, 89.1)
- added U7: TXS0102YZP, Package_BGA:Texas_DSBGA-8_0.9x1.9mm_Layout2x4_P0.5mm, F.Cu at (112.8, 121.6)
- added U8: TXS0102YZP, Package_BGA:Texas_DSBGA-8_0.9x1.9mm_Layout2x4_P0.5mm, F.Cu at (99.0, 92.1)
- added U9: BMX160, parts:PQFN50P250X300X100-14N, F.Cu at (144.7, 84.6)
- added Y1: 32.768k, Crystal:Crystal_SMD_2012-2Pin_2.0x1.2mm, F.Cu at (124.6, 121.9)
- added Y2: 32M, Crystal:Crystal_SMD_2012-2Pin_2.0x1.2mm, F.Cu at (134.5, 119.1)
- added Y3: 12M, Crystal:Crystal_SMD_2012-2Pin_2.0x1.2mm, F.Cu at (130.9, 119.1)
Other:
- copper layers 0 -> 2
