File: todd/hardware/todd_watch.kicad_sch (KiCad schematic)
At the start: 134 parts, among them J1 Expansion, J2 USB Device, J3 LRA, J4 Debug, J5 Strap, J6 Display, J7 Backlight, SW1 Up, SW2 Select, SW3 Down, SW4 Back, U1 NRF5340-QKAA-AB0-R, U2 MAX20353AEWN+, U3 TXS0102YZP, U4 TXS0102YZP, U5 TXS0102YZP, U6 BMX160, U7 S25FS512SDSBHV210, U8 Si1151-AB00, Y1 32.768k, Y2 32M

Commit message: Schem 1 done
Parts:
- removed J2: USB Device, Connector_USB:USB_C_Receptacle_XKB_U262-16XN-4BVC11, symbol Connector:USB_C_Receptacle_USB2.0
- removed J4: Debug, Connector_PinHeader_1.27mm:PinHeader_2x05_P1.27mm_Vertical, symbol Connector:Conn_ARM_JTAG_SWD_10
- removed JP9: SWD Power Reference, Connector_PinHeader_2.54mm:PinHeader_1x02_P2.54mm_Horizontal, symbol Jumper:Jumper_2_Bridged
- removed R5, R6: 5.1k, Resistor_SMD:R_0603_1608Metric, symbol Device:R
- added C38, C39: 27p, Capacitor_SMD:C_0603_1608Metric, symbol Device:C
- added C40, C41, C42, C43, C44, C45, C46: 100n, Capacitor_SMD:C_0603_1608Metric, symbol Device:C
- added J2: USB Device, symbol Connector_Generic:Conn_01x02
- added J4: USB Program, Connector_USB:USB_C_Receptacle_XKB_U262-16XN-4BVC11, symbol Connector:USB_C_Receptacle_USB2.0
- added J5: FTDI Flash, Connector_PinHeader_1.27mm:PinHeader_1x05_P1.27mm_Vertical, symbol Connector_Generic:Conn_01x05
- added R10: 10k, Resistor_SMD:R_0603_1608Metric, symbol Device:R
- added R11: 470, Resistor_SMD:R_0603_1608Metric, symbol Device:R
- added R7, R8: 5.1k, Resistor_SMD:R_0603_1608Metric, symbol Device:R
- added R9: 12k 1%, Resistor_SMD:R_0603_1608Metric, symbol Device:R
- added TP20: Hivolt SWDCLK, TestPoint:TestPoint_Pad_D1.0mm, symbol Connector:TestPoint
- added TP21: Hivolt SWDIO, TestPoint:TestPoint_Pad_D1.0mm, symbol Connector:TestPoint
- added TP22: Hivolt RESET, TestPoint:TestPoint_Pad_D1.0mm, symbol Connector:TestPoint
- added TP23: Spare Shift 3.3v, TestPoint:TestPoint_Pad_D1.0mm, symbol Connector:TestPoint
- added TP24: Spare Shift 1.8v, TestPoint:TestPoint_Pad_D1.0mm, symbol Connector:TestPoint
- added TP25: Lovolt SWDCLK, TestPoint:TestPoint_Pad_D1.0mm, symbol Connector:TestPoint
- added TP26: Lovolt SWDIO, TestPoint:TestPoint_Pad_D1.0mm, symbol Connector:TestPoint
- added TP27: Lovolt RESET, TestPoint:TestPoint_Pad_D1.0mm, symbol Connector:TestPoint
- added U3: FT232H, Package_QFP:LQFP-48_7x7mm_P0.5mm, symbol Interface_USB:FT232H
- added U4, U5: TXS0102YZP, Package_BGA:Texas_DSBGA-8_0.9x1.9mm_Layout2x4_P0.5mm, symbol Logic_LevelTranslator:TXS0102YZP
- added Y3: 12M, Crystal:Crystal_SMD_2012-2Pin_2.0x1.2mm, symbol Device:Crystal
- J1: footprint Connector_PinSocket_2.54mm:PinSocket_2x09_P2.54mm_Vertical -> Connector_PinSocket_1.27mm:PinSocket_2x09_P1.27mm_Vertical
- JP1, JP2, JP3, JP5, JP6: footprint Connector_PinHeader_2.54mm:PinHeader_1x02_P2.54mm_Horizontal -> Connector_PinHeader_1.27mm:PinHeader_2x01_P1.27mm_Horizontal
- JP10: renamed from JP11; footprint Connector_PinHeader_2.54mm:PinHeader_1x02_P2.54mm_Horizontal -> Connector_PinHeader_1.27mm:PinHeader_1x02_P1.27mm_Horizontal
- JP11: renamed from JP12; footprint Connector_PinHeader_2.54mm:PinHeader_1x02_P2.54mm_Horizontal -> Connector_PinHeader_1.27mm:PinHeader_1x02_P1.27mm_Horizontal
- JP13: renamed from JP14; footprint Connector_PinHeader_2.54mm:PinHeader_1x02_P2.54mm_Horizontal -> Connector_PinHeader_1.27mm:PinHeader_1x02_P1.27mm_Horizontal
- JP14: renamed from JP15; footprint Connector_PinHeader_2.54mm:PinHeader_1x02_P2.54mm_Horizontal -> Connector_PinHeader_1.27mm:PinHeader_1x02_P1.27mm_Horizontal
- JP15: renamed from JP16; footprint Connector_PinHeader_2.54mm:PinHeader_1x02_P2.54mm_Horizontal -> Connector_PinHeader_1.27mm:PinHeader_1x02_P1.27mm_Horizontal
- JP16: renamed from JP17; footprint Connector_PinHeader_2.54mm:PinHeader_1x02_P2.54mm_Horizontal -> Connector_PinHeader_1.27mm:PinHeader_1x02_P1.27mm_Horizontal
- JP17: renamed from JP18; footprint Connector_PinHeader_2.54mm:PinHeader_1x02_P2.54mm_Horizontal -> Connector_PinHeader_1.27mm:PinHeader_1x02_P1.27mm_Horizontal
- JP18: renamed from JP19; footprint Connector_PinHeader_2.54mm:PinHeader_1x02_P2.54mm_Horizontal -> Connector_PinHeader_1.27mm:PinHeader_1x02_P1.27mm_Horizontal
- JP7: renamed from JP8; footprint Connector_PinHeader_2.54mm:PinHeader_1x03_P2.54mm_Horizontal -> Connector_PinHeader_1.27mm:PinHeader_1x03_P1.27mm_Horizontal
- JP8: renamed from JP7; footprint Connector_PinHeader_2.54mm:PinHeader_1x03_P2.54mm_Horizontal -> Connector_PinHeader_1.27mm:PinHeader_1x03_P1.27mm_Horizontal
- JP9: renamed from JP10; footprint Connector_PinHeader_2.54mm:PinHeader_1x02_P2.54mm_Horizontal -> Connector_PinHeader_1.27mm:PinHeader_2x01_P1.27mm_Horizontal
- MK1: footprint MIC_ICS-40619 -> parts:MIC_ICS-40619
- TH1: footprint Connector_PinHeader_2.54mm:PinHeader_1x02_P2.54mm_Vertical -> Capacitor_SMD:C_0603_1608Metric
- U1: footprint XCVR_NRF5340-QKAA-AB0-R -> parts:XCVR_NRF5340-QKAA-AB0-R
- U10: renamed from U7; footprint FAB024_SPA -> parts:S25FL512SAGBHIC10
- U2: footprint 21-100104A_W563A4_1 -> parts:MAX20353AEWN&plus_
- U9: renamed from U6; footprint PQFN50P250X300X100-14N -> parts:PQFN50P250X300X100-14N
- Y1, Y2: footprint (none) -> Crystal:Crystal_SMD_2012-2Pin_2.0x1.2mm
- renumbered C38 to C47, C39 to C48, C40 to C49, C41 to C50, C42 to C51, C43 to C52, C44 to C53, J5 to J6, J6 to J7, J7 to J8, JP13 to JP12, R9 to R12, R10 to R13, R11 to R14, R7 to R2, R2 to R3, R3 to R4, R4 to R5, R8 to R6, TP7 to TP10, TP12 to TP11, TP13 to TP12, TP14 to TP13, TP15 to TP14, TP16 to TP15, TP17 to TP16, TP18 to TP17, TP19 to TP18, TP11 to TP19, TP20 to TP28, TP21 to TP29, TP22 to TP30, TP23 to TP31, TP8 to TP6, TP9 to TP7, TP10 to TP8, TP6 to TP9, U8 to U11, U3 to U6, U4 to U7, U5 to U8
Connections:
- net CPU_RESETn: now also TP27.1, U5.D2 (A1)
- net CPU_SWDCLK: now also TP25.1, U4.D2 (A1)
- net CPU_SWDIO: now also TP26.1, U4.D1 (A2)
- net CPU_USB_D+: now also J2.1 (Pin_1)
- net CPU_USB_D-: now also J2.2 (Pin_2)
- net GND: now also C38.1, C39.1, C40.1, C41.1, C42.1, C43.1, C44.1, C45.1, C46.1, J4.A1 (GND), J4.A12 (GND), J4.B1 (GND), J4.B12 (GND), J4.S1 (SHIELD), J5.1 (Pin_1), R7.2, R8.2, R9.1, U3.10 (GND), U3.11 (GND), U3.22 (GND), U3.23 (GND), U3.35 (GND), U3.36 (GND), U3.4 (AGND), U3.41 (AGND), U3.42 (TEST), U3.47 (GND), U3.48 (GND), U3.9 (AGND), U4.B1 (GND), U5.B1 (GND)
- net VBUS: now also J4.A4 (VBUS), J4.A9 (VBUS), J4.B4 (VBUS), J4.B9 (VBUS), U3.40 (VREGIN)
- new net: C42.2, C43.2, C44.2, C45.2, C46.2, J5.5 (Pin_5), R10.1, U3.12 (VCCIO), U3.24 (VCCIO), U3.3 (VPHY), U3.39 (VCCD), U3.46 (VCCIO), U3.8 (VPLL), U4.B2 (VCCB), U4.C2 (OE), U5.B2 (VCCB), U5.C2 (OE)
- new net: J4.B5 (CC2), R8.1
- new net: C40.2, U3.37 (VCCA)
- new net: TP23.1, U5.A1 (B2)
- new net: J4.A5 (CC1), R7.1
- new net: C38.2, U3.1 (XCSI), Y3.1
- new net: R11.1, U3.15 (ADBUS2)
- new net: C39.2, U3.2 (XCSO), Y3.2
- new net: R10.2, U3.34 (~{RESET})
- new net: C41.2, U3.38 (VCCCORE)
- new net: J5.2 (Pin_2), U3.43 (EEDATA)
- new net: J5.3 (Pin_3), U3.44 (EECLK)
- new net: J5.4 (Pin_4), U3.45 (EECS)
- new net: R9.2, U3.5 (REF)
- new net: U4.C1 (VCCA), U5.C1 (VCCA)
- new net: TP24.1, U5.D1 (A2)
- new net CPU_RESETn_HIVOLT: TP22.1, U3.18 (ADBUS5), U5.A2 (B1)
- new net CPU_SWDCLK_HIVOLT: TP20.1, U3.13 (ADBUS0), U4.A2 (B1)
- new net CPU_SWDIO_HIVOLT: R11.2, TP21.1, U3.14 (ADBUS1), U4.A1 (B2)
- new net FTDI_USB_D+: J4.A6 (D+), J4.B6 (D+), U3.7 (DP)
- new net FTDI_USB_D-: J4.A7 (D-), J4.B7 (D-), U3.6 (DM)
- no-connect marks 9 -> 21
Other:
- note added: ""Why all the jumpers" you might ask My plan is that I can use them to isolate parts of the board, so badly designed sections can be cut off and other sections tested independently"
- note added: "Buttons and Miscellany"
- note added: "Display"
- note added: "Don't know if I need eeprom for swd hope not"
- note added: "Just in case the FTDI doesn't work Backup debug pins both before and after the level shifters"
- note added: "Microcontroller"
- note added: "Peripherals"
- note added: "Power Regulation"
- note added: "Pretty sure I don't need these caps"
- note added: "Programming"
- note added: "This is because the first run of boards is gonna cost me $250 dollars, and if it doesn't work as a whole I'm gonna get my money's worth out of it one way or another"
- note removed: "Debug connector Note: watch expects 1.8v so use a genuine st-link or j-link that can handle it"
- note removed: "USB device signaling"
- note removed: "Will the final watch have a usb port? No Does the devkit? Yes Why? Dunno, might find a use for it"
- moved on the sheet: BT1, BT2, C23, C24, C25, C26, C27, C28, C29, C30, C31, C32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
